Commit message: Implement Ultra-Lightweight 2D Semantic Mapping with Zero-Stream WiFi mode

File: ros2_ws/src/robot_bringup/urdf/kobuki.urdf (robot description, URDF)
Before this commit: robot kobuki, 2 links, 1 joints
Links:
- added link camera_color_optical_frame
- added link camera_depth_optical_frame
Joints:
- added joint camera_color_optical_joint: type fixed, parent camera_link, child camera_color_optical_frame, origin xyz=0 0 0 rpy=-1.57079632679 0 -1.57079632679
- added joint camera_depth_optical_joint: type fixed, parent camera_link, child camera_depth_optical_frame, origin xyz=0 0 0 rpy=-1.57079632679 0 -1.57079632679
